Commit message: single robot xacro, configs and launch: spawn, state pub and bridge

File: description/robot/gazebo_control.xacro (robot description, xacro)
@@ -1,11 +1,12 @@
 <?xml version="1.0"?>
 <robot xmlns:xacro="http://www.ros.org/wiki/xacro">
-    <xacro:arg name="prefix" default="" />
+    <xacro:arg name="frame_prefix" default="artbot_" />
+    <xacro:arg name="topic_prefix" default="artbot/" />
     <gazebo>
         <plugin filename="ignition-gazebo-diff-drive-system"
         name="ignition::gazebo::systems::DiffDrive">
             <!-- Wheel Information -->
-            <left_joint>$(arg prefix)left_wheel_joint</left_joint>
-            <right_joint>$(arg prefix)right_wheel_joint</right_joint>
+            <left_joint>$(arg frame_prefix)left_wheel_joint</left_joint>
+            <right_joint>$(arg frame_prefix)right_wheel_joint</right_joint>
             <wheel_separation>0.297</wheel_separation>
             <wheel_radius>0.033</wheel_radius>
@@ -20,9 +21,9 @@
             <min_angular_velocity>-1</min_angular_velocity>
             <!-- Input -->
-            <topic>/$(arg prefix)cmd_vel</topic>
+            <topic>/$(arg topic_prefix)cmd_vel</topic>
             <!-- Output -->
-            <frame_id>$(arg prefix)odom</frame_id>
-            <child_frame_id>$(arg prefix)base_link</child_frame_id>
-            <odom_topic>/$(arg prefix)odom</odom_topic>
+            <frame_id>$(arg frame_prefix)odom</frame_id>
+            <child_frame_id>$(arg frame_prefix)base_link</child_frame_id>
+            <odom_topic>/$(arg topic_prefix)odom</odom_topic>
             <odom_publisher_frequency>30</odom_publisher_frequency>
             <tf_topic>/tf</tf_topic>
@@ -30,7 +31,7 @@
         <plugin filename="ignition-gazebo-joint-state-publisher-system"
             name="ignition::gazebo::systems::JointStatePublisher">
-            <topic>/$(arg prefix)joint_states</topic>
-            <joint_name>$(arg prefix)left_wheel_joint</joint_name>
-            <joint_name>$(arg prefix)right_wheel_joint</joint_name>
+            <topic>/$(arg topic_prefix)joint_states</topic>
+            <joint_name>$(arg frame_prefix)left_wheel_joint</joint_name>
+            <joint_name>$(arg frame_prefix)right_wheel_joint</joint_name>
         </plugin>
     </gazebo>

File: description/robot/lidar.xacro (robot description, xacro)
@@ -1,11 +1,12 @@
 <?xml version="1.0"?>
 <robot xmlns:xacro="http://www.ros.org/wiki/xacro" >
-    <xacro:arg name="prefix" default="" />
-    <joint name="$(arg prefix)laser_joint" type="fixed">
-        <parent link="$(arg prefix)chassis"/>
-        <child link="$(arg prefix)laser_frame"/>
+    <xacro:arg name="frame_prefix" default="artbot_" />
+    <xacro:arg name="topic_prefix" default="artbot/" />
+    <joint name="$(arg frame_prefix)laser_joint" type="fixed">
+        <parent link="$(arg frame_prefix)chassis"/>
+        <child link="$(arg frame_prefix)laser_frame"/>
         <origin xyz="0.122 0 0.212" rpy="0 0 0"/>
     </joint>
-    <link name="$(arg prefix)laser_frame">
+    <link name="$(arg frame_prefix)laser_frame">
         <visual>
             <geometry>
@@ -30,7 +31,7 @@
         </xacro:inertial_cylinder>
     </link>
-    <gazebo reference="$(arg prefix)laser_frame">
+    <gazebo reference="$(arg frame_prefix)laser_frame">
         <material>Gazebo/Black</material>
-        <sensor name="$(arg prefix)laser" type="gpu_lidar">
+        <sensor name="$(arg frame_prefix)laser" type="gpu_lidar">
             <pose> 0 0 0 0 0 0 </pose>
             <visualize>false</visualize>
@@ -49,6 +50,6 @@
                 </range>
             </lidar>
-            <topic>/$(arg prefix)scan</topic>
-            <gz_frame_id>$(arg prefix)laser_frame</gz_frame_id>
+            <topic>/$(arg topic_prefix)scan</topic>
+            <gz_frame_id>$(arg frame_prefix)laser_frame</gz_frame_id>
         </sensor>
     </gazebo>

File: description/robot/robot.urdf.xacro (robot description, xacro)
@@ -1,5 +1,6 @@
 <?xml version="1.0"?>
 <robot xmlns:xacro="http://www.ros.org/wiki/xacro"  name="articulate_bot">
-    <xacro:arg name="prefix" default="" />
+    <xacro:arg name="frame_prefix" default="artbot_" />
+    <xacro:arg name="topic_prefix" default="artbot/" />
     <xacro:include filename="robot_core.xacro"/>
     <xacro:include filename="gazebo_control.xacro"/>

File: description/robot/robot_core.xacro (robot description, xacro)
@@ -1,5 +1,6 @@
 <?xml version="1.0"?>
 <robot xmlns:xacro="http://www.ros.org/wiki/xacro" >
-    <xacro:arg name="prefix" default="" />
+    <xacro:arg name="frame_prefix" default="artbot_" />
+    <xacro:arg name="topic_prefix" default="artbot/" />
     <xacro:include filename="inertial_macros.xacro"/>
     <xacro:property name="chassis_length" value="0.335"/>
@@ -33,21 +34,21 @@
     </material>
     <!-- BASE LINK -->
-    <link name="$(arg prefix)base_link">
+    <link name="$(arg frame_prefix)base_link">
     </link>
     <!-- BASE_FOOTPRINT LINK -->
-    <joint name="$(arg prefix)base_footprint_joint" type="fixed">
-        <parent link="$(arg prefix)base_link"/>
-        <child link="$(arg prefix)base_footprint"/>
+    <joint name="$(arg frame_prefix)base_footprint_joint" type="fixed">
+        <parent link="$(arg frame_prefix)base_link"/>
+        <child link="$(arg frame_prefix)base_footprint"/>
         <origin xyz="0 0 0" rpy="0 0 0"/>
     </joint>
-    <link name="$(arg prefix)base_footprint">
+    <link name="$(arg frame_prefix)base_footprint">
     </link>
     <!-- CHASSIS LINK -->
-    <joint name="$(arg prefix)chassis_joint" type="fixed">
-        <parent link="$(arg prefix)base_link"/>
-        <child link="$(arg prefix)chassis"/>
+    <joint name="$(arg frame_prefix)chassis_joint" type="fixed">
+        <parent link="$(arg frame_prefix)base_link"/>
+        <child link="$(arg frame_prefix)chassis"/>
         <origin xyz="${-wheel_offset_x} 0 ${-wheel_offset_z}"/>
     </joint>
-    <link name="$(arg prefix)chassis">
+    <link name="$(arg frame_prefix)chassis">
         <visual>
             <origin xyz="${chassis_length/2} 0 ${chassis_height/2}"/>
@@ -67,15 +68,15 @@
         </xacro:inertial_box>
     </link>
-    <gazebo reference="$(arg prefix)chassis">
+    <gazebo reference="$(arg frame_prefix)chassis">
         <material>Gazebo/Orange</material>
     </gazebo>
     <!-- LEFT WHEEL LINK -->
-    <joint name="$(arg prefix)left_wheel_joint" type="continuous">
-        <parent link="$(arg prefix)base_link"/>
-        <child link="$(arg prefix)left_wheel"/>
+    <joint name="$(arg frame_prefix)left_wheel_joint" type="continuous">
+        <parent link="$(arg frame_prefix)base_link"/>
+        <child link="$(arg frame_prefix)left_wheel"/>
         <origin xyz="0 ${wheel_offset_y} 0" rpy="-${pi/2} 0 0" />
         <axis xyz="0 0 1"/>
     </joint>
-    <link name="$(arg prefix)left_wheel">
+    <link name="$(arg frame_prefix)left_wheel">
         <visual>
             <geometry>
@@ -93,15 +94,15 @@
         </xacro:inertial_cylinder>
     </link>
-    <gazebo reference="$(arg prefix)left_wheel">
+    <gazebo reference="$(arg frame_prefix)left_wheel">
         <material>Gazebo/Blue</material>
     </gazebo>
     <!-- RIGHT WHEEL LINK -->
-    <joint name="$(arg prefix)right_wheel_joint" type="continuous">
-        <parent link="$(arg prefix)base_link"/>
-        <child link="$(arg prefix)right_wheel"/>
+    <joint name="$(arg frame_prefix)right_wheel_joint" type="continuous">
+        <parent link="$(arg frame_prefix)base_link"/>
+        <child link="$(arg frame_prefix)right_wheel"/>
         <origin xyz="0 ${-wheel_offset_y} 0" rpy="${pi/2} 0 0" />
         <axis xyz="0 0 -1"/>
     </joint>
-    <link name="$(arg prefix)right_wheel">
+    <link name="$(arg frame_prefix)right_wheel">
         <visual>
             <geometry>
@@ -119,14 +120,14 @@
         </xacro:inertial_cylinder>
     </link>
-    <gazebo reference="$(arg prefix)right_wheel">
+    <gazebo reference="$(arg frame_prefix)right_wheel">
         <material>Gazebo/Blue</material>
     </gazebo>
     <!-- CASTER WHEEL LINK -->
-    <joint name="$(arg prefix)caster_wheel_joint" type="fixed">
-        <parent link="$(arg prefix)chassis"/>
-        <child link="$(arg prefix)caster_wheel"/>
+    <joint name="$(arg frame_prefix)caster_wheel_joint" type="fixed">
+        <parent link="$(arg frame_prefix)chassis"/>
+        <child link="$(arg frame_prefix)caster_wheel"/>
         <origin xyz="${caster_wheel_offset_x} 0 ${caster_wheel_offset_z}"/>
     </joint>
-    <link name="$(arg prefix)caster_wheel">
+    <link name="$(arg frame_prefix)caster_wheel">
         <visual>
             <geometry>
@@ -144,5 +145,5 @@
         </xacro:inertial_sphere>
     </link>
-    <gazebo reference="$(arg prefix)caster_wheel">
+    <gazebo reference="$(arg frame_prefix)caster_wheel">
         <material>Gazebo/White</material>
         <mu1 value="0.001"/>
